File: hw/XassetteAsterisk.kicad_pcb (KiCad board)
At the start: 2 copper layers, 56 x 56 mm, 133 parts, among them J1 Conn_01x40_MountingPin, J10 Conn_02x03_Odd_Even, J11 Conn_01x02, J12 Conn_01x03, J2 Conn_01x24_MountingPin, J3 AudioJack4, J4 USB4105-GF-A, J5 USB4105-GF-A, J6 AudioJack4, J7 Conn_01x04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

Commit message: hw upgrade to v0.2
Parts:
- removed R22, R23, R34: 10k, Resistor_SMD:R_0603_1608Metric
- removed R24: 1.5k, Resistor_SMD:R_0603_1608Metric
- removed the RST at (113.7, 151.8)
- added C59: 0.1u, Capacitor_SMD:C_0603_1608Metric, B.Cu at (123.3, 138.9)
- added D10: ESD9B3.3ST5G, Diode_SMD:D_SOD-923, B.Cu at (111.0, 107.2)
- added D11: ESD9B3.3ST5G, Diode_SMD:D_SOD-923, B.Cu at (112.4, 107.2)
- added D12: ESD9B3.3ST5G, Diode_SMD:D_SOD-923, B.Cu at (126.0, 107.2)
- added D13: ESD9B3.3ST5G, Diode_SMD:D_SOD-923, B.Cu at (124.7, 107.2)
- added D5: ESD9B3.3ST5G, Diode_SMD:D_SOD-923, B.Cu at (143.1, 108.1)
- added D6: ESD9B3.3ST5G, Diode_SMD:D_SOD-923, B.Cu at (141.6, 108.1)
- added D7: ESD9B3.3ST5G, Diode_SMD:D_SOD-923, B.Cu at (138.4, 108.1)
- added D8: ESD9B3.3ST5G, Diode_SMD:D_SOD-923, B.Cu at (136.8, 108.1)
- added D9: ESD9B3.3ST5G, Diode_SMD:D_SOD-923, B.Cu at (140.0, 108.1)
- added FEL: SW_SPST, Button_Switch_SMD:SW_SPST_EVQPE1, F.Cu at (111.1, 152.7)
- added J13: RTL8189FTV_Mod, 8189ftvMod:8189Mod, F.Cu at (114.4, 143.4)
- added RN2: R_Pack04, Resistor_SMD:R_Array_Convex_4x0603, F.Cu at (109.0, 135.5)
- added RST: SW_SPST, Button_Switch_SMD:SW_SPST_EVQPE1, F.Cu at (118.1, 152.7)
- C1, C13, C14, C5: value 0.1u -> 18p
- C46: value 0.1u -> 10u
- J10: footprint Connector_PinHeader_2.54mm:PinHeader_2x03_P2.54mm_Vertical -> Connector_PinHeader_2.00mm:PinHeader_2x03_P2.00mm_Vertical
- R1, R2, R3: value 1.5k -> 5.1k
- R11: value 100k -> 10k
- R12: value 100k -> 5.1k
- R20: value 1k -> 100k
- R9: value 1k -> 10M
- moved R12 9.53 mm to (113.5, 135.9)
- moved R14 3.41 mm to (113.5, 132.0)
- moved R16 3.39 mm to (116.9, 132.0)
- moved C7 2.50 mm to (116.9, 127.0)
- moved C9 2.49 mm to (116.9, 129.5)
- moved R21 1.74 mm to (112.8, 141.2)
- moved R18 1.60 mm to (110.5, 141.2)
- moved J10 1.26 mm to (124.8, 116.2)
- moved R4 1.03 mm to (112.9, 145.6)
- moved U2 1.00 mm to (117.4, 142.8)
- moved C57 0.82 mm to (116.4, 138.9)
- moved R17 0.76 mm to (110.5, 145.6), turned to 90 degrees
- moved C54 0.76 mm to (148.1, 108.2)
- moved D3 0.39 mm to (116.9, 135.9)
- moved U5 0.14 mm to (110.3, 129.4)
- renumbered PE to JP1, PD to JP2, PG to JP3
Connections:
- R12 pad 1: Net-(C12-Pad1) -> +3V3
- R12 pad 2: GND -> Net-(D3-Pad2)
Routing:
- net +3V3: track 270.1 -> 329.0 mm, vias 12 -> 13
- net /PC5: track 28.9 -> 39.8 mm
- net /PC7: track 38.3 -> 48.6 mm, vias 2 -> 4
- net /PC2: track 33.6 -> 39.8 mm, vias 1 -> 2
- net Net-(C43-Pad1): track 3.10 -> 8.80 mm, vias 0 -> 1
- net Net-(C42-Pad1): track 8.25 -> 13.1 mm, vias 0 -> 1
- net /VDD-CORE: track 83.0 -> 87.8 mm
- net /PC4: track 35.4 -> 39.6 mm, vias 1 -> 2
- net /PC6: track 28.8 -> 32.2 mm
- net /HS_MIC: track 11.2 -> 14.5 mm, vias 1 -> 2
- net Net-(R14-Pad1): track 4.39 -> 7.65 mm
- net +5V: track 204.2 -> 207.4 mm
- net Net-(C12-Pad1): track 28.8 -> 25.7 mm, vias 5 -> 4
- net /PC3: track 43.0 -> 40.5 mm
- net /RST: track 27.8 -> 30.1 mm
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
Commit message: hw upgrade to v0.3
Parts:
- added R22: 5.1k, Resistor_SMD:R_0603_1608Metric, B.Cu at (118.6, 107.8)
- added R23: 5.1k, Resistor_SMD:R_0603_1608Metric, B.Cu at (118.5, 105.5)
- added R24: 5.1k, Resistor_SMD:R_0603_1608Metric, B.Cu at (118.5, 102.9)
- renumbered FEL to FEL1, RST to RST1
Connections:
- C55 pad 1: +3V3 -> GND
- C55 pad 2: GND -> +3V3
- J2 pad 23: +3V3 -> /CSI-IOVDD
- J2 pad 24: +3V3 -> /CSI-IOVDD
- JP1 pad 2: /VCC_PE -> /CSI-IOVDD
- U1 pad 34: /VCC_PE -> /CSI-IOVDD
Routing:
- net /CSI-IOVDD: track 0.00 -> 42.2 mm, vias 0 -> 2
- net +3V3: track 329.0 -> 299.7 mm, vias 13 -> 12
- net Net-(J4-PadB5): track 0.00 -> 12.0 mm, vias 0 -> 1
- net Net-(J5-PadB5): track 0.00 -> 9.63 mm, vias 0 -> 1
- net /VCC_PE: track 4.74 -> 0.00 mm, vias 1 -> 0
- net +5V: track 207.4 -> 210.4 mm, vias 5 -> 6
