File: hw/XassetteAsterisk.sch (KiCad schematic (older format))
At the start: 132 parts, among them J1 Conn_01x40_MountingPin, J10 Conn_02x03_Odd_Even, J11 Conn_01x02, J12 Conn_01x03, J2 Conn_01x24_MountingPin, J3 AudioJack4, J4 USB4105-GF-A, J5 USB4105-GF-A, J6 AudioJack4, J7 Conn_01x04, J8 Conn_02x17_Odd_Even, J9 Conn_01x06, SW1 SW_SPST, U1 F133, U2 W25Q32JVSS, U3 SY8089AAAC, U4 SY8089AAAC, U5 SY8089AAAC, U6 SY7201ABC, U7 XC6206PxxxMR, Y1 Crystal, Y2 24M

Commit message: schematic revision
Parts:
- C1, C5: value 0.1u -> 18p
- C13, C14: value 0.1u -> 30p
- C46: value 0.1u -> 10u
- R11: value 100k -> 10k
- R12: value 100k -> NC
- R20: value 1k -> 100k
- R9: value 1k -> 10M
Changed lines of the file:
@@
 $EndComp
 $Comp
-L Device:C C1
-U 1 1 6166B949
-P 5550 5750
-F 0 "C1" V 5298 5750 50  0000 C CNN
-F 1 "0.1u" V 5389 5750 50  0000 C CNN
-F 2 "Capacitor_SMD:C_0603_1608Metric" H 5588 5600 50  0001 C CNN
-F 3 "~" H 5550 5750 50  0001 C CNN
-	1    5550 5750
-	0    1    1    0
-$EndComp
-$Comp
-L Device:C C5
-U 1 1 6166E38F
-P 5550 6150
-F 0 "C5" V 5298 6150 50  0000 C CNN
-F 1 "0.1u" V 5389 6150 50  0000 C CNN
-F 2 "Capacitor_SMD:C_0603_1608Metric" H 5588 6000 50  0001 C CNN
-F 3 "~" H 5550 6150 50  0001 C CNN
-	1    5550 6150
-	0    1    1    0
-$EndComp
-$Comp
 L Device:R R9
 U 1 1 6166E82F
 P 6250 5950
 F 0 "R9" H 6150 5900 50  0000 C CNN
-F 1 "1k" H 6150 6000 50  0000 C CNN
+F 1 "10M" H 6150 6000 50  0000 C CNN
 F 2 "Resistor_SMD:R_0603_1608Metric" V 6180 5950 50  0001 C CNN
 F 3 "~" H 6250 5950 50  0001 C CNN
@@
 P 1300 8400
 F 0 "R11" H 1200 8350 50  0000 C CNN
-F 1 "100k" H 1150 8450 50  0000 C CNN
+F 1 "10k" H 1150 8450 50  0000 C CNN
 F 2 "Resistor_SMD:R_0603_1608Metric" V 1230 8400 50  0001 C CNN
 F 3 "~" H 1300 8400 50  0001 C CNN
@@
 P 1300 8800
 F 0 "R12" H 1200 8750 50  0000 C CNN
-F 1 "100k" H 1150 8850 50  0000 C CNN
+F 1 "NC" H 1150 8850 50  0000 C CNN
 F 2 "Resistor_SMD:R_0603_1608Metric" V 1230 8800 50  0001 C CNN
 F 3 "~" H 1300 8800 50  0001 C CNN
@@
 P 5700 4400
 F 0 "C14" V 5448 4400 50  0000 C CNN
-F 1 "0.1u" V 5539 4400 50  0000 C CNN
+F 1 "30p" V 5539 4400 50  0000 C CNN
 F 2 "Capacitor_SMD:C_0603_1608Metric" H 5738 4250 50  0001 C CNN
 F 3 "~" H 5700 4400 50  0001 C CNN
@@
 P 5400 5150
 F 0 "C13" V 5148 5150 50  0000 C CNN
-F 1 "0.1u" V 5239 5150 50  0000 C CNN
+F 1 "30p" V 5239 5150 50  0000 C CNN
 F 2 "Capacitor_SMD:C_0603_1608Metric" H 5438 5000 50  0001 C CNN
 F 3 "~" H 5400 5150 50  0001 C CNN
@@
 U 1 1 61A47327
 P 4450 6400
-F 0 "R20" H 4350 6350 50  0000 C CNN
-F 1 "1k" H 4350 6450 50  0000 C CNN
+F 0 "R20" H 4300 6350 50  0000 C CNN
+F 1 "100k" H 4300 6450 50  0000 C CNN
 F 2 "Resistor_SMD:R_0603_1608Metric" V 4380 6400 50  0001 C CNN
 F 3 "~" H 4450 6400 50  0001 C CNN
@@
 P 1050 3000
 F 0 "C46" V 798 3000 50  0000 C CNN
-F 1 "0.1u" V 889 3000 50  0000 C CNN
+F 1 "10u" V 889 3000 50  0000 C CNN
 F 2 "Capacitor_SMD:C_0603_1608Metric" H 1088 2850 50  0001 C CNN
 F 3 "~" H 1050 3000 50  0001 C CNN
@@
 Wire Wire Line
 	7350 2850 7350 3100
+$Comp
+L Device:C C5
+U 1 1 6166E38F
+P 5550 6150
+F 0 "C5" V 5298 6150 50  0000 C CNN
+F 1 "18p" V 5389 6150 50  0000 C CNN
+F 2 "Capacitor_SMD:C_0603_1608Metric" H 5588 6000 50  0001 C CNN
+F 3 "~" H 5550 6150 50  0001 C CNN
+	1    5550 6150
+	0    1    1    0
+$EndComp
+$Comp
+L Device:C C1
+U 1 1 6166B949
+P 5550 5750
+F 0 "C1" V 5298 5750 50  0000 C CNN
+F 1 "18p" V 5389 5750 50  0000 C CNN
+F 2 "Capacitor_SMD:C_0603_1608Metric" H 5588 5600 50  0001 C CNN
+F 3 "~" H 5550 5750 50  0001 C CNN
+	1    5550 5750
+	0    1    1    0
+$EndComp
 $EndSCHEMATC

Commit message: minor changes in schematic
Parts:
- C13, C14: value 30p -> 18p
- R1, R2, R3: value 1.5k -> 5.1k
Changed lines of the file:
@@
 P 5700 4400
 F 0 "C14" V 5448 4400 50  0000 C CNN
-F 1 "30p" V 5539 4400 50  0000 C CNN
+F 1 "18p" V 5539 4400 50  0000 C CNN
 F 2 "Capacitor_SMD:C_0603_1608Metric" H 5738 4250 50  0001 C CNN
 F 3 "~" H 5700 4400 50  0001 C CNN
@@
 P 5400 5150
 F 0 "C13" V 5148 5150 50  0000 C CNN
-F 1 "30p" V 5239 5150 50  0000 C CNN
+F 1 "18p" V 5239 5150 50  0000 C CNN
 F 2 "Capacitor_SMD:C_0603_1608Metric" H 5438 5000 50  0001 C CNN
 F 3 "~" H 5400 5150 50  0001 C CNN
@@
 P 11300 1100
 F 0 "R1" V 11200 950 50  0000 C CNN
-F 1 "1.5k" V 11200 1200 50  0000 C CNN
+F 1 "5.1k" V 11200 1200 50  0000 C CNN
 F 2 "Resistor_SMD:R_0603_1608Metric" V 11230 1100 50  0001 C CNN
 F 3 "~" H 11300 1100 50  0001 C CNN
@@
 P 11700 1100
 F 0 "R2" V 11600 950 50  0000 C CNN
-F 1 "1.5k" V 11650 1250 50  0000 C CNN
+F 1 "5.1k" V 11650 1250 50  0000 C CNN
 F 2 "Resistor_SMD:R_0603_1608Metric" V 11630 1100 50  0001 C CNN
 F 3 "~" H 11700 1100 50  0001 C CNN
@@
 P 13900 1300
 F 0 "R3" H 13800 1350 50  0000 C CNN
-F 1 "1.5k" H 13800 1450 50  0000 C CNN
+F 1 "5.1k" H 13800 1450 50  0000 C CNN
 F 2 "Resistor_SMD:R_0603_1608Metric" V 13830 1300 50  0001 C CNN
 F 3 "~" H 13900 1300 50  0001 C CNN

Commit message: hw upgrade to v0.2
Parts:
- removed R22, R23, R34: 10k, Resistor_SMD:R_0603_1608Metric, symbol Device:R
- removed R24: 1.5k, Resistor_SMD:R_0603_1608Metric, symbol Device:R
- added C59: 0.1u, Capacitor_SMD:C_0603_1608Metric, symbol Device:C
- added D10, D11, D12, D13, D5, D6, D7, D8, D9: ESD9B3.3ST5G, Diode_SMD:D_SOD-923, symbol Diode:ESD9B3.3ST5G
- added FEL1: SW_SPST, Button_Switch_SMD:SW_SPST_EVQPE1, symbol Switch:SW_SPST
- added J13: RTL8189FTV_Mod, 8189ftvMod:8189Mod, symbol Connector_Generic:Conn_02x07_Counter_Clockwise
- added RN2: R_Pack04, Resistor_SMD:R_Array_Convex_4x0603, symbol Device:R_Pack04
- J10: footprint Connector_PinHeader_2.54mm:PinHeader_2x03_P2.54mm_Vertical -> Connector_PinHeader_2.00mm:PinHeader_2x03_P2.00mm_Vertical
- R12: value NC -> 5.1k
- RST1: renamed from SW1; footprint Button_Switch_SMD:SW_SPST_FSMSM -> Button_Switch_SMD:SW_SPST_EVQPE1
Connections:
- net +3V3: now also R12.1, C59.1, J13.11 (Pin_11), J13.12 (Pin_12), J13.13 (Pin_13), RN2.1 (R1.1), RN2.2 (R2.1), RN2.3 (R3.1)
- net GND: now also C59.2, D10.1 (A1), D11.1 (A1), D12.1 (A1), D13.1 (A1), D5.1 (A1), D6.1 (A1), D7.1 (A1), D8.1 (A1), D9.1 (A1), FEL1.1 (A), J13.7 (Pin_7), J13.8 (Pin_8), RN2.4 (R4.1), RN2.5 (R4.2); no longer R12.2
- net HS_MIC: now also D9.2 (A2)
- net PC2: now also J13.6 (Pin_6)
- net PC3: now also J13.1 (Pin_1), RN2.8 (R1.2)
- net PC4: now also J13.3 (Pin_3)
- net PC5: now also FEL1.2 (B), J13.4 (Pin_4)
- net PC6: now also J13.5 (Pin_5)
- net PC7: now also J13.2 (Pin_2)
- net PF3: now also RN2.6 (R3.2)
- net PF6: now also RN2.7 (R2.2)
- net USB0_N: now also D11.2 (A2)
- net USB0_P: now also D10.2 (A2)
- net USB1_N: now also D13.2 (A2)
- net USB1_P: now also D12.2 (A2)
- net at C12.1, R11.2, U4.1 (EN)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: no longer R12.1
- net at D3.2 (A): now also R12.2
- net at C47.1, J6.R1: now also D8.2 (A2)
- net at C48.1, J6.T: now also D7.2 (A2)
- net at C42.1, J3.R1: now also D6.2 (A2)
- net at C43.1, J3.T: now also D5.2 (A2)
- no-connect marks 9 -> 11
Other:
- note added: "FEL button"
- moved on the sheet: C13, C14, C23, C35, C36, C37, C42, C43, C47, C48, C50, C51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

Commit message: hw upgrade to v0.3
Parts:
- added R22, R23, R24: 5.1k, Resistor_SMD:R_0603_1608Metric, symbol Device:R
Connections:
- net +3V3: now also C55.2; no longer C55.1, J2.23 (Pin_23), J2.24 (Pin_24)
- net +5V: now also R23.1, R24.1
- net GND: now also C55.1, R22.2; no longer C55.2
- net at J4.B5 (CC2): now also R22.1, R23.2
- net at J5.B5 (CC2): now also R24.2
- net VCC_PE renamed CSI-IOVDD
- net CSI-IOVDD: now also J2.23 (Pin_23), J2.24 (Pin_24)
- no-connect marks 11 -> 9
Other:
- moved on the sheet: C1, C10, C11, C12, C13, C14, C15, C16, C17, C18, C19, C2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
